Commit message: add velocity limits

File: st_r17_description/urdf/robot_3.urdf (robot description, URDF)
Before this commit: robot st_r17, 7 links, 6 joints
Joints:
- joint elbow: limit (none) -> effort=1000.0 velocity=2.26
- joint hand: limit (none) -> effort=1000.0 velocity=5.58
- joint shoulder: axis 0 0 1 -> 0 0 -1; child link_2 -> link_1; limit (none) -> effort=1000.0 velocity=1.57; origin xyz=0 0 0.32173 rpy=1.5708 1.5708 3.1416 -> xyz=0 0 0.033268 rpy=-6.123E-17 0 0; parent link_1 -> base_link
- joint waist: limit lower=-3.1 upper=3.1 effort=1000.0 velocity=0.5 -> lower=-3.1 upper=3.1 effort=1000.0 velocity=2.6
- joint wrist: limit (none) -> effort=1000.0 velocity=5.58

Commit message: fixed srange error

File: st_r17_description/urdf/robot_3.urdf (robot description, URDF)
Before this commit: robot st_r17, 7 links, 6 joints
Joints:
- joint shoulder: axis 0 0 -1 -> 0 0 1; child link_1 -> link_2; origin xyz=0 0 0.033268 rpy=-6.123E-17 0 0 -> xyz=0 0 0.32173 rpy=1.5708 1.5708 3.1416; parent base_link -> link_1
