Commit message: adding reasonable stereo camera

File: st_r17_description/urdf/robot.urdf.xacro (robot description, xacro)
@@ -1,5 +1,7 @@
 <robot name="st_r17" xmlns:xacro="http://ros.org/wiki/xacro">
+	<xacro:include filename="$(find st_r17_description)/urdf/stereo.urdf.xacro"/>
 	<xacro:property name="deg" value="${pi/180.0}"/>
     <xacro:arg name="use_kinect" default="true"/>
+    <xacro:arg name="use_stereo" default="true"/>
 	<xacro:macro name="box_inertia" params="x y z mass">
 		<inertia ixx="${0.0833333 * mass * (y*y + z*z)}" ixy="0.0" ixz="0.0"
@@ -437,4 +439,15 @@
         </plugin>
     </gazebo>
+    <!-- Stereo -->
+    <xacro:if value="$(arg use_stereo)">
+        <link name="stereo_link"> </link>
+        <joint name="stereo_joint" type="fixed">
+            <origin xyz="0.15875 0 0.012"/>
+            <parent link="link_5"/>
+            <child link="stereo_link"/>
+            <axis xyz="0 0 1"/>
+        </joint>
+        <xacro:stereo baseline="0.0636" parent="stereo_link"/>
+    </xacro:if>
     <!-- Kinect -->
     <xacro:if value="$(arg use_kinect)">

Commit message: working dh calibration ... consider separating these out

File: st_r17_description/urdf/robot.urdf.xacro (robot description, xacro)
@@ -446,4 +446,11 @@
             <parent link="link_5"/>
             <child link="stereo_link"/>
+            <axis xyz="0 0 1"/>
+        </joint>
+        <link name="stereo_optical_link"> </link>
+        <joint name="stereo_optical_joint" type="fixed">
+            <origin xyz="0 0 0" rpy="${-pi/2} 0 ${-pi/2}"/>
+            <parent link="stereo_link"/>
+            <child link="stereo_optical_link"/>
             <axis xyz="0 0 1"/>
         </joint>

Commit message: now detecting april tags in gazebo; fairly close to a working dh calibration!

File: st_r17_description/urdf/robot.urdf.xacro (robot description, xacro)
@@ -9,4 +9,9 @@
 			izz="${0.0833333 * mass * (x*x + y*y)}" />
 	</xacro:macro>
+    <link name="world"/>
+    <joint name="fixed" type="fixed">
+        <parent link="world"/>
+        <child link="base_link"/>
+    </joint>
 	<link
 		name="base_link">
